Commit message: Imported files form ur_description & robotiq_description into ur10e_description; Edited files to always look for ur10e_description
This was done to avoid problems with values in the ur_desccription and
robotiq_description packages not being editable (Such as for the problem
with initial position!)

This might not be the optimal way to fix this, but it's nice that
everything is self-contained now

File: ur10e_description/urdf/robotiq_2f_85_urdf.xacro (robot description, xacro)
@@ -4,4 +4,5 @@
     <xacro:arg name="use_fake_hardware" default="false" />
     <xacro:arg name="sim_ignition" default="true" />
+    <xacro:arg name="name" default="robotiq_gripper"/>
     <!-- If visualizing just the gripper with no arm, set the true, otherwise, set to false -->
     <xacro:property name="gripper_only" value="false"/>
@@ -18,5 +19,5 @@
         com_port:=/dev/ttyUSB0">
         <!-- ros2 control include -->
-        <xacro:include filename="$(find robotiq_description)/urdf/robotiq_gripper.ros2_control.xacro" />
+        <xacro:include filename="$(find ur10e_description)/urdf/robotiq_gripper.ros2_control.xacro" />
         <!-- if we are simulating or directly communicating with the gripper we need a ros2 control instance -->
         <xacro:if value="${include_ros2_control}">
@@ -32,10 +33,10 @@
             <visual>
                 <geometry>
-                    <mesh filename="file://$(find robotiq_description)/meshes/visual/robotiq_base.dae" />
-                </geometry>
-            </visual>
-            <collision>
-                <geometry>
-                    <mesh filename="file://$(find robotiq_description)/meshes/collision/robotiq_base.stl" />
+                    <mesh filename="file://$(find ur10e_description)/meshes/$(arg name)/visual/robotiq_base.dae" />
+                </geometry>
+            </visual>
+            <collision>
+                <geometry>
+                    <mesh filename="file://$(find ur10e_description)/meshes/$(arg name)/collision/robotiq_base.stl" />
                 </geometry>
             </collision>
@@ -49,10 +50,10 @@
             <visual>
                 <geometry>
-                    <mesh filename="file://$(find robotiq_description)/meshes/visual/left_knuckle.dae" />
-                </geometry>
-            </visual>
-            <collision>
-                <geometry>
-                    <mesh filename="file://$(find robotiq_description)/meshes/collision/left_knuckle.stl" />
+                    <mesh filename="file://$(find ur10e_description)/meshes/$(arg name)/visual/left_knuckle.dae" />
+                </geometry>
+            </visual>
+            <collision>
+                <geometry>
+                    <mesh filename="file://$(find ur10e_description)/meshes/$(arg name)/collision/left_knuckle.stl" />
                 </geometry>
             </collision>
@@ -66,10 +67,10 @@
             <visual>
                 <geometry>
-                    <mesh filename="file://$(find robotiq_description)/meshes/visual/right_knuckle.dae" />
-                </geometry>
-            </visual>
-            <collision>
-                <geometry>
-                    <mesh filename="file://$(find robotiq_description)/meshes/collision/right_knuckle.stl" />
+                    <mesh filename="file://$(find ur10e_description)/meshes/$(arg name)/visual/right_knuckle.dae" />
+                </geometry>
+            </visual>
+            <collision>
+                <geometry>
+                    <mesh filename="file://$(find ur10e_description)/meshes/$(arg name)/collision/right_knuckle.stl" />
                 </geometry>
             </collision>
@@ -83,10 +84,10 @@
             <visual>
                 <geometry>
-                    <mesh filename="file://$(find robotiq_description)/meshes/visual/left_finger.dae" />
-                </geometry>
-            </visual>
-            <collision>
-                <geometry>
-                    <mesh filename="file://$(find robotiq_description)/meshes/collision/left_finger.stl" />
+                    <mesh filename="file://$(find ur10e_description)/meshes/$(arg name)/visual/left_finger.dae" />
+                </geometry>
+            </visual>
+            <collision>
+                <geometry>
+                    <mesh filename="file://$(find ur10e_description)/meshes/$(arg name)/collision/left_finger.stl" />
                 </geometry>
             </collision>
@@ -100,10 +101,10 @@
             <visual>
                 <geometry>
-                    <mesh filename="file://$(find robotiq_description)/meshes/visual/right_finger.dae" />
-                </geometry>
-            </visual>
-            <collision>
-                <geometry>
-                    <mesh filename="file://$(find robotiq_description)/meshes/collision/right_finger.stl" />
+                    <mesh filename="file://$(find ur10e_description)/meshes/$(arg name)/visual/right_finger.dae" />
+                </geometry>
+            </visual>
+            <collision>
+                <geometry>
+                    <mesh filename="file://$(find ur10e_description)/meshes/$(arg name)/collision/right_finger.stl" />
                 </geometry>
             </collision>
@@ -117,10 +118,10 @@
             <visual>
                 <geometry>
-                    <mesh filename="file://$(find robotiq_description)/meshes/visual/left_inner_knuckle.dae" />
-                </geometry>
-            </visual>
-            <collision>
-                <geometry>
-                    <mesh filename="file://$(find robotiq_description)/meshes/collision/left_inner_knuckle.stl" />
+                    <mesh filename="file://$(find ur10e_description)/meshes/$(arg name)/visual/left_inner_knuckle.dae" />
+                </geometry>
+            </visual>
+            <collision>
+                <geometry>
+                    <mesh filename="file://$(find ur10e_description)/meshes/$(arg name)/collision/left_inner_knuckle.stl" />
                 </geometry>
             </collision>
@@ -134,10 +135,10 @@
             <visual>
                 <geometry>
-                    <mesh filename="file://$(find robotiq_description)/meshes/visual/right_inner_knuckle.dae" />
-                </geometry>
-            </visual>
-            <collision>
-                <geometry>
-                    <mesh filename="file://$(find robotiq_description)/meshes/collision/right_inner_knuckle.stl" />
+                    <mesh filename="file://$(find ur10e_description)/meshes/$(arg name)/visual/right_inner_knuckle.dae" />
+                </geometry>
+            </visual>
+            <collision>
+                <geometry>
+                    <mesh filename="file://$(find ur10e_description)/meshes/$(arg name)/collision/right_inner_knuckle.stl" />
                 </geometry>
             </collision>
@@ -151,10 +152,10 @@
             <visual>
                 <geometry>
-                    <mesh filename="file://$(find robotiq_description)/meshes/visual/left_finger_tip.dae" />
-                </geometry>
-            </visual>
-            <collision>
-                <geometry>
-                    <mesh filename="file://$(find robotiq_description)/meshes/collision/left_finger_tip.stl" />
+                    <mesh filename="file://$(find ur10e_description)/meshes/$(arg name)/visual/left_finger_tip.dae" />
+                </geometry>
+            </visual>
+            <collision>
+                <geometry>
+                    <mesh filename="file://$(find ur10e_description)/meshes/$(arg name)/collision/left_finger_tip.stl" />
                 </geometry>
                 <surface>
@@ -186,10 +187,10 @@
             <visual>
                 <geometry>
-                    <mesh filename="file://$(find robotiq_description)/meshes/visual/right_finger_tip.dae" />
-                </geometry>
-            </visual>
-            <collision>
-                <geometry>
-                    <mesh filename="file://$(find robotiq_description)/meshes/collision/right_finger_tip.stl" />
+                    <mesh filename="file://$(find ur10e_description)/meshes/$(arg name)/visual/right_finger_tip.dae" />
+                </geometry>
+            </visual>
+            <collision>
+                <geometry>
+                    <mesh filename="file://$(find ur10e_description)/meshes/$(arg name)/collision/right_finger_tip.stl" />
                 </geometry>
                 <surface>

File: ur10e_description/urdf/ur10e_urdf.xacro (robot description, xacro)
@@ -6,5 +6,5 @@
    <xacro:arg name="name" default="ur"/>
    <!-- import main macro -->
-   <xacro:include filename="$(find ur_description)/urdf/ur_macro.xacro"/>
+   <xacro:include filename="$(find ur10e_description)/urdf/ur_macro.xacro"/>
    <!-- possible 'ur_type' values: ur3, ur10e, ur5, ur5e, ur10, ur10e, ur16e, ur20, ur30 -->
    <!-- the default value should raise an error in case this was called without defining the type -->
@@ -12,8 +12,8 @@
    <!-- parameters -->
    <xacro:arg name="tf_prefix" default="ur10e_" />
-   <xacro:arg name="joint_limit_params" default="$(find ur_description)/config/$(arg ur_type)/joint_limits.yaml"/>
-   <xacro:arg name="kinematics_params" default="$(find ur_description)/config/$(arg ur_type)/default_kinematics.yaml"/>
-   <xacro:arg name="physical_params" default="$(find ur_description)/config/$(arg ur_type)/physical_parameters.yaml"/>
-   <xacro:arg name="visual_params" default="$(find ur_description)/config/$(arg ur_type)/visual_parameters.yaml"/>
+   <xacro:arg name="joint_limit_params" default="$(find ur10e_description)/config/joint_limits.yaml"/>
+   <xacro:arg name="kinematics_params" default="$(find ur10e_description)/config/default_kinematics.yaml"/>
+   <xacro:arg name="physical_params" default="$(find ur10e_description)/config/physical_parameters.yaml"/>
+   <xacro:arg name="visual_params" default="$(find ur10e_description)/config/visual_parameters.yaml"/>
    <xacro:arg name="transmission_hw_interface" default=""/>
    <xacro:arg name="safety_limits" default="false"/>
@@ -48,5 +48,5 @@
    <xacro:arg name="simulation_controllers" default="$(arg controllers_config_file)" /> <!-- Controllers copied from UR ROS2 Driver Package -->
    <!-- initial position for simulations (Fake Hardware, Gazebo, Ignition) -->
-   <xacro:arg name="initial_positions_file" default="$(find ur_description)/config/initial_positions.yaml"/>
+   <xacro:arg name="initial_positions_file" default="$(find ur10e_description)/config/initial_positions.yaml"/>
    <!-- convert to property to use substitution in function -->
    <xacro:property name="initial_positions_file" default="$(arg initial_positions_file)"/>

Commit message: Edited urdf files to fix issue w/ meshes not loading in Gazebo

File: ur10e_description/urdf/robotiq_2f_85_urdf.xacro (robot description, xacro)
@@ -4,5 +4,4 @@
     <xacro:arg name="use_fake_hardware" default="false" />
     <xacro:arg name="sim_ignition" default="true" />
-    <xacro:arg name="name" default="robotiq_gripper"/>
     <!-- If visualizing just the gripper with no arm, set the true, otherwise, set to false -->
     <xacro:property name="gripper_only" value="false"/>
@@ -33,10 +32,10 @@
             <visual>
                 <geometry>
-                    <mesh filename="file://$(find ur10e_description)/meshes/$(arg name)/visual/robotiq_base.dae" />
-                </geometry>
-            </visual>
-            <collision>
-                <geometry>
-                    <mesh filename="file://$(find ur10e_description)/meshes/$(arg name)/collision/robotiq_base.stl" />
+                    <mesh filename="file://$(find ur10e_description)/meshes/robotiq_gripper/visual/robotiq_base.dae" />
+                </geometry>
+            </visual>
+            <collision>
+                <geometry>
+                    <mesh filename="file://$(find ur10e_description)/meshes/robotiq_gripper/collision/robotiq_base.stl" />
                 </geometry>
             </collision>
@@ -50,10 +49,10 @@
             <visual>
                 <geometry>
-                    <mesh filename="file://$(find ur10e_description)/meshes/$(arg name)/visual/left_knuckle.dae" />
-                </geometry>
-            </visual>
-            <collision>
-                <geometry>
-                    <mesh filename="file://$(find ur10e_description)/meshes/$(arg name)/collision/left_knuckle.stl" />
+                    <mesh filename="file://$(find ur10e_description)/meshes/robotiq_gripper/visual/left_knuckle.dae" />
+                </geometry>
+            </visual>
+            <collision>
+                <geometry>
+                    <mesh filename="file://$(find ur10e_description)/meshes/robotiq_gripper/collision/left_knuckle.stl" />
                 </geometry>
             </collision>
@@ -67,10 +66,10 @@
             <visual>
                 <geometry>
-                    <mesh filename="file://$(find ur10e_description)/meshes/$(arg name)/visual/right_knuckle.dae" />
-                </geometry>
-            </visual>
-            <collision>
-                <geometry>
-                    <mesh filename="file://$(find ur10e_description)/meshes/$(arg name)/collision/right_knuckle.stl" />
+                    <mesh filename="file://$(find ur10e_description)/meshes/robotiq_gripper/visual/right_knuckle.dae" />
+                </geometry>
+            </visual>
+            <collision>
+                <geometry>
+                    <mesh filename="file://$(find ur10e_description)/meshes/robotiq_gripper/collision/right_knuckle.stl" />
                 </geometry>
             </collision>
@@ -84,10 +83,10 @@
             <visual>
                 <geometry>
-                    <mesh filename="file://$(find ur10e_description)/meshes/$(arg name)/visual/left_finger.dae" />
-                </geometry>
-            </visual>
-            <collision>
-                <geometry>
-                    <mesh filename="file://$(find ur10e_description)/meshes/$(arg name)/collision/left_finger.stl" />
+                    <mesh filename="file://$(find ur10e_description)/meshes/robotiq_gripper/visual/left_finger.dae" />
+                </geometry>
+            </visual>
+            <collision>
+                <geometry>
+                    <mesh filename="file://$(find ur10e_description)/meshes/robotiq_gripper/collision/left_finger.stl" />
                 </geometry>
             </collision>
@@ -101,10 +100,10 @@
             <visual>
                 <geometry>
-                    <mesh filename="file://$(find ur10e_description)/meshes/$(arg name)/visual/right_finger.dae" />
-                </geometry>
-            </visual>
-            <collision>
-                <geometry>
-                    <mesh filename="file://$(find ur10e_description)/meshes/$(arg name)/collision/right_finger.stl" />
+                    <mesh filename="file://$(find ur10e_description)/meshes/robotiq_gripper/visual/right_finger.dae" />
+                </geometry>
+            </visual>
+            <collision>
+                <geometry>
+                    <mesh filename="file://$(find ur10e_description)/meshes/robotiq_gripper/collision/right_finger.stl" />
                 </geometry>
             </collision>
@@ -118,10 +117,10 @@
             <visual>
                 <geometry>
-                    <mesh filename="file://$(find ur10e_description)/meshes/$(arg name)/visual/left_inner_knuckle.dae" />
-                </geometry>
-            </visual>
-            <collision>
-                <geometry>
-                    <mesh filename="file://$(find ur10e_description)/meshes/$(arg name)/collision/left_inner_knuckle.stl" />
+                    <mesh filename="file://$(find ur10e_description)/meshes/robotiq_gripper/visual/left_inner_knuckle.dae" />
+                </geometry>
+            </visual>
+            <collision>
+                <geometry>
+                    <mesh filename="file://$(find ur10e_description)/meshes/robotiq_gripper/collision/left_inner_knuckle.stl" />
                 </geometry>
             </collision>
@@ -135,10 +134,10 @@
             <visual>
                 <geometry>
-                    <mesh filename="file://$(find ur10e_description)/meshes/$(arg name)/visual/right_inner_knuckle.dae" />
-                </geometry>
-            </visual>
-            <collision>
-                <geometry>
-                    <mesh filename="file://$(find ur10e_description)/meshes/$(arg name)/collision/right_inner_knuckle.stl" />
+                    <mesh filename="file://$(find ur10e_description)/meshes/robotiq_gripper/visual/right_inner_knuckle.dae" />
+                </geometry>
+            </visual>
+            <collision>
+                <geometry>
+                    <mesh filename="file://$(find ur10e_description)/meshes/robotiq_gripper/collision/right_inner_knuckle.stl" />
                 </geometry>
             </collision>
@@ -152,10 +151,10 @@
             <visual>
                 <geometry>
-                    <mesh filename="file://$(find ur10e_description)/meshes/$(arg name)/visual/left_finger_tip.dae" />
-                </geometry>
-            </visual>
-            <collision>
-                <geometry>
-                    <mesh filename="file://$(find ur10e_description)/meshes/$(arg name)/collision/left_finger_tip.stl" />
+                    <mesh filename="file://$(find ur10e_description)/meshes/robotiq_gripper/visual/left_finger_tip.dae" />
+                </geometry>
+            </visual>
+            <collision>
+                <geometry>
+                    <mesh filename="file://$(find ur10e_description)/meshes/robotiq_gripper/collision/left_finger_tip.stl" />
                 </geometry>
                 <surface>
@@ -187,10 +186,10 @@
             <visual>
                 <geometry>
-                    <mesh filename="file://$(find ur10e_description)/meshes/$(arg name)/visual/right_finger_tip.dae" />
-                </geometry>
-            </visual>
-            <collision>
-                <geometry>
-                    <mesh filename="file://$(find ur10e_description)/meshes/$(arg name)/collision/right_finger_tip.stl" />
+                    <mesh filename="file://$(find ur10e_description)/meshes/robotiq_gripper/visual/right_finger_tip.dae" />
+                </geometry>
+            </visual>
+            <collision>
+                <geometry>
+                    <mesh filename="file://$(find ur10e_description)/meshes/robotiq_gripper/collision/right_finger_tip.stl" />
                 </geometry>
                 <surface>

File: ur10e_description/urdf/robotiq_gripper.ros2_control.xacro (robot description, xacro)
@@ -38,5 +38,5 @@
                 <command_interface name="position" />
                 <state_interface name="position">
-                    <param name="initial_value">0.7929</param>
+                    <param name="initial_value">0</param>
                 </state_interface>
                 <state_interface name="velocity"/>

File: ur10e_description/urdf/ur.ros2_control.xacro (robot description, xacro)
@@ -7,5 +7,5 @@
     sim_ignition:=false
     headless_mode:=false
-    initial_positions:=${dict(shoulder_pan_joint=0.0,shoulder_lift_joint=-1.57,elbow_joint=0.0,wrist_1_joint=-1.57,wrist_2_joint=0.0,wrist_3_joint=0.0)}
+    initial_positions:=${dict(shoulder_pan_joint=0.0,shoulder_lift_joint=0,elbow_joint=0.0,wrist_1_joint=0,wrist_2_joint=0.0,wrist_3_joint=0.0)}
     use_tool_communication:=false
     script_filename output_recipe_filename
